Commit message: archive

File: markhor_description/urdf/kinova_common.xacro (robot description, xacro)
@@ -39,4 +39,40 @@
     </link>
   </xacro:macro>
+  <xacro:macro name="flipper_link" params="link_name link_mesh link_origin_xyz:='0 0 0' link_origin_rpy:='0 0 0' link_material:='red' has_collision_mesh:=false">
+    <link name="${link_name}">
+      <visual>
+        <geometry>
+          <mesh filename="package://markhor_description/meshes/visual/${link_mesh}.stl"/>
+        </geometry>
+        <origin xyz="${link_origin_xyz}" rpy="${link_origin_rpy}"/>
+        <material name="${link_material}"/>
+      </visual>
+      <collision>
+        <geometry>
+          <xacro:if value="${has_collision_mesh}">
+            <mesh filename="package://markhor_description/meshes/collision/${link_mesh}.stl"/>
+          </xacro:if>
+          <xacro:unless value="${has_collision_mesh}">
+            <mesh filename="package://markhor_description/meshes/visual/${link_mesh}.stl"/>
+          </xacro:unless>
+        </geometry>
+        <origin xyz="${link_origin_xyz}" rpy="${link_origin_rpy}"/>
+        <surface>
+          <friction>
+            <ode>
+              <mu>0.7</mu>
+              <mu2>150</mu2>
+              <fdir1>0 1 0</fdir1>
+            </ode>
+          </friction>
+          <contact>
+            <ode/>
+          </contact>
+        </surface>
+      </collision>
+      <max_contacts>20</max_contacts>
+      <xacro:markhor_inertial link_name="${link_name}"/>
+    </link>
+  </xacro:macro>
   <xacro:macro name="kinova_joint" params="joint_name type parent child joint_axis_xyz joint_origin_xyz joint_origin_rpy joint_lower_limit joint_upper_limit joint_velocity_limit joint_torque_limit fixed:=false">
     <joint name="${joint_name}" type="${type}">
@@ -72,4 +108,60 @@
     </xacro:unless>
   </xacro:macro>
+  <xacro:macro name="flipper_joint" params="joint_name type parent child joint_axis_xyz joint_origin_xyz joint_origin_rpy joint_lower_limit joint_upper_limit joint_velocity_limit joint_torque_limit fixed:=false">
+    <joint name="${joint_name}" type="${type}">
+      <parent link="${parent}"/>
+      <child link="${child}"/>
+      <axis xyz="${joint_axis_xyz}"/>
+      <limit effort="${joint_torque_limit}" velocity="${joint_velocity_limit}" lower="${joint_lower_limit}" upper="${joint_upper_limit}"/>
+      <origin xyz="${joint_origin_xyz}" rpy="${joint_origin_rpy}"/>
+      <dynamics damping="0.0" friction="0.0"/>
+      <physics>
+        <ode>
+          <implicit_spring_damper>1</implicit_spring_damper>
+          <cfm_damping>1</cfm_damping>
+          <limit>
+            <cfm>0</cfm>
+            <erp>0.2</erp>
+          </limit>
+        </ode>
+      </physics>
+    </joint>
+    <xacro:unless value="${fixed}">
+      <transmission name="${joint_name}_trans">
+        <type>transmission_interface/SimpleTransmission</type>
+        <joint name="${joint_name}">
+          <hardwareInterface>hardware_interface/EffortJointInterface</hardwareInterface>
+        </joint>
+        <actuator name="${joint_name}_actuator">
+          <hardwareInterface>hardware_interface/EffortJointInterface</hardwareInterface>
+          <mechanicalReduction>1</mechanicalReduction>
+        </actuator>
+      </transmission>
+    </xacro:unless>
+  </xacro:macro>
+  <xacro:macro name="track_joint" params="joint_name type parent child joint_axis_xyz joint_origin_xyz joint_origin_rpy joint_velocity_limit joint_torque_limit fixed:=false">
+    <joint name="${joint_name}" type="${type}">
+      <parent link="${parent}"/>
+      <child link="${child}"/>
+      <axis xyz="${joint_axis_xyz}"/>
+      <limit effort="${joint_torque_limit}" velocity="${joint_velocity_limit}"/>
+      <origin xyz="${joint_origin_xyz}" rpy="${joint_origin_rpy}"/>
+      <dynamics damping="0.0" friction="0.0"/>
+      <physics>
+        <ode/>
+      </physics>
+    </joint>
+    <xacro:unless value="${fixed}">
+      <transmission name="${joint_name}_trans">
+        <type>transmission_interface/SimpleTransmission</type>
+        <joint name="${joint_name}">
+          <hardwareInterface>hardware_interface/VelocityJointInterface</hardwareInterface>
+        </joint>
+        <actuator name="${joint_name}_motor">
+          <mechanicalReduction>1</mechanicalReduction>
+        </actuator>
+      </transmission>
+    </xacro:unless>
+  </xacro:macro>
   <xacro:macro name="kinova_virtual_link" params="link_name">
     <link name="${link_name}"/>
@@ -84,19 +176,3 @@
     </joint>
   </xacro:macro>
-  <xacro:macro name="sim_wheel" params="wheel_name wheel_rad wheel_width wheel_parent">
-    <link name="${wheel_name}_link">
-      <visual>
-        <geometry>
-          <cylinder length="${wheel_width}" radius="${wheel_rad}"/>
-        </geometry>
-        <origin xyz="0 0 0" rpy="0 ${pi/2} 0"/>
-        <material name="white"/>
-      </visual>
-    </link>
-    <joint name="${wheel_name}_joint" type="continuous">
-      <parent link="${wheel_parent}"/>
-      <child link="${wheel_name}_link"/>
-      <axis xyz="1 0 0"/>
-    </joint>
-  </xacro:macro>
 </root>

File: markhor_description/urdf/markhor.xacro (robot description, xacro)
@@ -130,20 +130,4 @@
     <xacro:property name="joint_lidar_origin_xyz" value="0.32034017 0 -0.1393156" />
     <xacro:property name="joint_lidar_origin_rpy" value="${pi} 0 0" />
-    <!-- FL Wheel -->
-    <xacro:property name="fl_wheel_name" value="fl_wheel"/>
-    <xacro:property name="fl_wheel_rad" value="0.1318"/>
-    <xacro:property name="fl_wheel_width" value="0.12065"/>
-    <!-- FR Wheel -->
-    <xacro:property name="fr_wheel_name" value="fr_wheel"/>
-    <xacro:property name="fr_wheel_rad" value="0.1318"/>
-    <xacro:property name="fr_wheel_width" value="0.12065"/>
-    <!-- RL Wheel -->
-    <xacro:property name="rl_wheel_name" value="rl_wheel"/>
-    <xacro:property name="rl_wheel_rad" value="0.1318"/>
-    <xacro:property name="rl_wheel_width" value="0.12065"/>
-    <!-- RR Wheel -->
-    <xacro:property name="rr_wheel_name" value="rr_wheel"/>
-    <xacro:property name="rr_wheel_rad" value="0.1318"/>
-    <xacro:property name="rr_wheel_width" value="0.12065"/>
     <xacro:macro name="markhor" params="base_parent prefix:=markhor">
         <xacro:kinova_link link_name="${prefix}_link_base" link_mesh="${link_base_mesh}" link_origin_rpy="${link_base_origin_rpy}"/>
@@ -158,12 +142,16 @@
         <xacro:kinova_joint joint_name="${prefix}_joint_gb_rr" type="${joint_gb_rr_type}" parent="${prefix}_link_base" child="${prefix}_link_gb_rr" joint_axis_xyz="${joint_gb_rr_axis_xyz}" joint_origin_xyz="${joint_gb_rr_origin_xyz}" joint_origin_rpy="${joint_gb_rr_origin_rpy}" joint_lower_limit="0" joint_upper_limit="0" joint_velocity_limit="0" joint_torque_limit="0" fixed="true"/>
         <!-- flipper angle frame -->
-        <xacro:kinova_link link_name="${prefix}_link_flip_fl" link_mesh="${link_flip_fl_mesh}" link_material="${link_flip_material}"/>
-        <xacro:kinova_joint joint_name="${prefix}_joint_flip_fl" type="${joint_flip_fl_type}" parent="${prefix}_link_gb_fl" child="${prefix}_link_flip_fl" joint_axis_xyz="${joint_flip_fl_axis_xyz}" joint_origin_xyz="${joint_flip_fl_origin_xyz}" joint_origin_rpy="${joint_flip_fl_origin_rpy}" joint_lower_limit="${joint_flip_fl_lower_limit}" joint_upper_limit="${joint_flip_fl_upper_limit}" joint_velocity_limit="${joint_flip_fl_velocity_limit}" joint_torque_limit="${joint_flip_fl_torque_limit}"/>
-        <xacro:kinova_link link_name="${prefix}_link_flip_fr" link_mesh="${link_flip_fr_mesh}" link_material="${link_flip_material}"/>
-        <xacro:kinova_joint joint_name="${prefix}_joint_flip_fr" type="${joint_flip_fr_type}" parent="${prefix}_link_gb_fr" child="${prefix}_link_flip_fr" joint_axis_xyz="${joint_flip_fr_axis_xyz}" joint_origin_xyz="${joint_flip_fr_origin_xyz}" joint_origin_rpy="${joint_flip_fr_origin_rpy}" joint_lower_limit="${joint_flip_fr_lower_limit}" joint_upper_limit="${joint_flip_fr_upper_limit}" joint_velocity_limit="${joint_flip_fr_velocity_limit}" joint_torque_limit="${joint_flip_fr_torque_limit}"/>
-        <xacro:kinova_link link_name="${prefix}_link_flip_rl" link_mesh="${link_flip_rl_mesh}" link_material="${link_flip_material}"/>
-        <xacro:kinova_joint joint_name="${prefix}_joint_flip_rl" type="${joint_flip_rl_type}" parent="${prefix}_link_gb_rl" child="${prefix}_link_flip_rl" joint_axis_xyz="${joint_flip_rl_axis_xyz}" joint_origin_xyz="${joint_flip_rl_origin_xyz}" joint_origin_rpy="${joint_flip_rl_origin_rpy}" joint_lower_limit="${joint_flip_rl_lower_limit}" joint_upper_limit="${joint_flip_rl_upper_limit}" joint_velocity_limit="${joint_flip_rl_velocity_limit}" joint_torque_limit="${joint_flip_rl_torque_limit}"/>
-        <xacro:kinova_link link_name="${prefix}_link_flip_rr" link_mesh="${link_flip_rr_mesh}" link_material="${link_flip_material}"/>
-        <xacro:kinova_joint joint_name="${prefix}_joint_flip_rr" type="${joint_flip_rr_type}" parent="${prefix}_link_gb_rr" child="${prefix}_link_flip_rr" joint_axis_xyz="${joint_flip_rr_axis_xyz}" joint_origin_xyz="${joint_flip_rr_origin_xyz}" joint_origin_rpy="${joint_flip_rr_origin_rpy}" joint_lower_limit="${joint_flip_rr_lower_limit}" joint_upper_limit="${joint_flip_rr_upper_limit}" joint_velocity_limit="${joint_flip_rr_velocity_limit}" joint_torque_limit="${joint_flip_rr_torque_limit}"/>
+        <xacro:flipper_link link_name="${prefix}_link_flip_fl" link_mesh="${link_flip_fl_mesh}" link_material="${link_flip_material}"/>
+        <xacro:flipper_joint joint_name="${prefix}_joint_flip_fl" type="${joint_flip_fl_type}" parent="${prefix}_link_gb_fl" child="${prefix}_link_flip_fl" joint_axis_xyz="${joint_flip_fl_axis_xyz}" joint_origin_xyz="${joint_flip_fl_origin_xyz}" joint_origin_rpy="${joint_flip_fl_origin_rpy}" joint_lower_limit="${joint_flip_fl_lower_limit}" joint_upper_limit="${joint_flip_fl_upper_limit}" joint_velocity_limit="${joint_flip_fl_velocity_limit}" joint_torque_limit="${joint_flip_fl_torque_limit}"/>
+        <!-- <xacro:track_joint joint_name="${prefix}_joint_track_fl" type="${joint_track_fl_type}" parent="${prefix}_link_gb_fl" child="${prefix}_link_flip_fl" joint_axis_xyz="${joint_flip_fl_axis_xyz}" joint_origin_xyz="${joint_flip_fl_origin_xyz}" joint_origin_rpy="${joint_flip_fl_origin_rpy}" joint_velocity_limit="${joint_track_fl_velocity_limit}" joint_torque_limit="${joint_track_fl_torque_limit}"/> -->
+        <xacro:flipper_link link_name="${prefix}_link_flip_fr" link_mesh="${link_flip_fr_mesh}" link_material="${link_flip_material}"/>
+        <xacro:flipper_joint joint_name="${prefix}_joint_flip_fr" type="${joint_flip_fr_type}" parent="${prefix}_link_gb_fr" child="${prefix}_link_flip_fr" joint_axis_xyz="${joint_flip_fr_axis_xyz}" joint_origin_xyz="${joint_flip_fr_origin_xyz}" joint_origin_rpy="${joint_flip_fr_origin_rpy}" joint_lower_limit="${joint_flip_fr_lower_limit}" joint_upper_limit="${joint_flip_fr_upper_limit}" joint_velocity_limit="${joint_flip_fr_velocity_limit}" joint_torque_limit="${joint_flip_fr_torque_limit}"/>
+        <!-- <xacro:track_joint joint_name="${prefix}_joint_track_fr" type="${joint_track_fl_type}" parent="${prefix}_link_gb_fl" child="${prefix}_link_flip_fr" joint_axis_xyz="${joint_flip_fl_axis_xyz}" joint_origin_xyz="${joint_flip_fl_origin_xyz}" joint_origin_rpy="${joint_flip_fl_origin_rpy}" joint_velocity_limit="${joint_track_fl_velocity_limit}" joint_torque_limit="${joint_track_fl_torque_limit}"/> -->
+        <xacro:flipper_link link_name="${prefix}_link_flip_rl" link_mesh="${link_flip_rl_mesh}" link_material="${link_flip_material}"/>
+        <xacro:flipper_joint joint_name="${prefix}_joint_flip_rl" type="${joint_flip_rl_type}" parent="${prefix}_link_gb_rl" child="${prefix}_link_flip_rl" joint_axis_xyz="${joint_flip_rl_axis_xyz}" joint_origin_xyz="${joint_flip_rl_origin_xyz}" joint_origin_rpy="${joint_flip_rl_origin_rpy}" joint_lower_limit="${joint_flip_rl_lower_limit}" joint_upper_limit="${joint_flip_rl_upper_limit}" joint_velocity_limit="${joint_flip_rl_velocity_limit}" joint_torque_limit="${joint_flip_rl_torque_limit}"/>
+        <!-- <xacro:track_joint joint_name="${prefix}_joint_track_rl" type="${joint_track_fl_type}" parent="${prefix}_link_gb_fl" child="${prefix}_link_flip_rl" joint_axis_xyz="${joint_flip_fl_axis_xyz}" joint_origin_xyz="${joint_flip_fl_origin_xyz}" joint_origin_rpy="${joint_flip_fl_origin_rpy}" joint_velocity_limit="${joint_track_fl_velocity_limit}" joint_torque_limit="${joint_track_fl_torque_limit}"/> -->
+        <xacro:flipper_link link_name="${prefix}_link_flip_rr" link_mesh="${link_flip_rr_mesh}" link_material="${link_flip_material}"/>
+        <xacro:flipper_joint joint_name="${prefix}_joint_flip_rr" type="${joint_flip_rr_type}" parent="${prefix}_link_gb_rr" child="${prefix}_link_flip_rr" joint_axis_xyz="${joint_flip_rr_axis_xyz}" joint_origin_xyz="${joint_flip_rr_origin_xyz}" joint_origin_rpy="${joint_flip_rr_origin_rpy}" joint_lower_limit="${joint_flip_rr_lower_limit}" joint_upper_limit="${joint_flip_rr_upper_limit}" joint_velocity_limit="${joint_flip_rr_velocity_limit}" joint_torque_limit="${joint_flip_rr_torque_limit}"/>
+        <!-- <xacro:track_joint joint_name="${prefix}_joint_track_rr" type="${joint_track_fl_type}" parent="${prefix}_link_gb_fl" child="${prefix}_link_flip_rr" joint_axis_xyz="${joint_flip_fl_axis_xyz}" joint_origin_xyz="${joint_flip_fl_origin_xyz}" joint_origin_rpy="${joint_flip_fl_origin_rpy}" joint_velocity_limit="${joint_track_fl_velocity_limit}" joint_torque_limit="${joint_track_fl_torque_limit}"/> -->
         <!-- Anchor for the front camera -->
         <xacro:kinova_virtual_link link_name="${prefix}_link_front_cam"/>
@@ -183,10 +171,8 @@
         <robotNamespace>$(arg robot_namespace)</robotNamespace>
       </plugin>
-    </gazebo>
-    <gazebo>
-      <plugin name="imu_controller" filename="libhector_gazebo_ros_imu.so">
+      <!-- <plugin name="imu_controller" filename="libhector_gazebo_ros_imu.so">
         <robotNamespace>$(arg robot_namespace)</robotNamespace>
         <updateRate>50.0</updateRate>
-        <bodyName>base_link</bodyName>
+        <bodyName>${prefix}_link_base</bodyName>
         <topicName>imu/data</topicName>
         <accelDrift>0.005 0.005 0.005</accelDrift>
@@ -196,5 +182,22 @@
         <headingDrift>0.005</headingDrift>
         <headingGaussianNoise>0.005</headingGaussianNoise>
+      </plugin> -->
+      <plugin filename="libSimpleTrackedVehiclePlugin.so" name="simple_tracked_vehicle">
+        <body>markhor_root</body>
+        <left_track>markhor_link_flip_fl</left_track>
+        <right_track>markhor_link_flip_fr</right_track>
+        <left_flipper>markhor_link_flip_rl</left_flipper>
+        <right_flipper>markhor_link_flip_rr</right_flipper>
+        <max_linear_speed>100</max_linear_speed>
+        <track_mu>2</track_mu>
+        <track_mu2>0.5</track_mu2>
       </plugin>
+      <!-- <plugin filename="libKeysToCmdVelPlugin.so" name="keyboard_control">
+        <publish_as_twist>true</publish_as_twist>
+        <cmd_vel_topic>~/markhor/cmd_vel_twist</cmd_vel_topic>
+        <max_linear_vel>100</max_linear_vel>
+        <min_linear_vel>-100</min_linear_vel>
+        <linear_increment>50</linear_increment>
+      </plugin> -->
     </gazebo>
 </root>

File: markhor_description/urdf/markhor_inertial.xacro (robot description, xacro)
@@ -17,5 +17,5 @@
         <xacro:if value="${link_name == 'markhor_link_base'}">
             <inertial>
-                <mass value="16.111" />
+                <mass value="1.5" />
                 <origin xyz="-0.00002529 0.00000008 -0.06049447" rpy="0 0 0"/>
                 <inertia ixx="0.385006414" ixy="0.0000696244868" ixz="-0.000181517937" iyy="0.624959190" iyz="0.000000162897534" izz="0.798949961"/>
@@ -25,5 +25,5 @@
         <xacro:if value="${link_name == 'markhor_link_gb_fl'}">
             <inertial>
-                <mass value="2.5"/>
+                <mass value="0.1"/>
                 <origin xyz="0.038 -0.038 0.014" rpy="0 0 0"/>
                 <inertia ixx="6.06448598e-2" ixy="1.93186915e-4" ixz="-1.57873663e-5" iyy="1.82869143e-2" iyz="2.81755463e-3" izz="5.13408129e-2"/>
@@ -33,5 +33,5 @@
         <xacro:if value="${link_name == 'markhor_link_gb_fr'}">
             <inertial>
-                <mass value="2.5"/>
+                <mass value="0.1"/>
                 <origin xyz="-0.038 -0.038 0.014" rpy="0 0 0"/>
                 <inertia ixx="6.06448598e-2" ixy="-1.93186915e-4" ixz="1.57873663e-5" iyy="1.82869143e-2" iyz="2.81755463e-3" izz="5.13408129e-2"/>
@@ -41,5 +41,5 @@
         <xacro:if value="${link_name == 'markhor_link_gb_rl'}">
             <inertial>
-                <mass value="2.5"/>
+                <mass value="0.1"/>
                 <origin xyz="-0.038 -0.038 0.014" rpy="0 0 0"/>
                 <inertia ixx="6.06448598e-2" ixy="-1.93186915e-4" ixz="1.57873663e-5" iyy="1.82869143e-2" iyz="2.81755463e-3" izz="5.13408129e-2"/>
@@ -49,5 +49,5 @@
         <xacro:if value="${link_name == 'markhor_link_gb_rr'}">
             <inertial>
-                <mass value="2.5"/>
+                <mass value="0.1"/>
                 <origin xyz="0.038 -0.038 0.014" rpy="0 0 0"/>
                 <inertia ixx="6.06448598e-2" ixy="1.93186915e-4" ixz="-1.57873663e-5" iyy="1.82869143e-2" iyz="2.81755463e-3" izz="5.13408129e-2"/>
@@ -57,5 +57,5 @@
         <xacro:if value="${link_name == 'markhor_link_flip_fl'}">
             <inertial>
-                <mass value="6.9"/>
+                <mass value="0.6"/>
                 <origin xyz="0 0.116 0" rpy="0 0 0"/>
                 <inertia ixx="0.268046334" ixy="0.000960466048" ixz="0.000262590776" iyy="0.0573569235" iyz="0.0000904647719" izz="0.232597105"/>
@@ -65,5 +65,5 @@
         <xacro:if value="${link_name == 'markhor_link_flip_fr'}">
             <inertial>
-                <mass value="6.9"/>
+                <mass value="0.6"/>
                 <origin xyz="0 0.116 0" rpy="0 0 0"/>
                 <inertia ixx="0.268046334" ixy="0.000960466048" ixz="0.000262590776" iyy="0.0573569235" iyz="0.0000904647719" izz="0.232597105"/>
@@ -73,5 +73,5 @@
         <xacro:if value="${link_name == 'markhor_link_flip_rl'}">
             <inertial>
-                <mass value="6.9"/>
+                <mass value="0.6"/>
                 <origin xyz="0 0.116 0" rpy="0 0 0"/>
                 <inertia ixx="0.268046334" ixy="0.000960466048" ixz="0.000262590776" iyy="0.0573569235" iyz="0.0000904647719" izz="0.232597105"/>
@@ -81,5 +81,5 @@
         <xacro:if value="${link_name == 'markhor_link_flip_rr'}">
             <inertial>
-                <mass value="6.9"/>
+                <mass value="0.6"/>
                 <origin xyz="0 0.116 0" rpy="0 0 0"/>
                 <inertia ixx="0.268046334" ixy="0.000960466048" ixz="0.000262590776" iyy="0.0573569235" iyz="0.0000904647719" izz="0.232597105"/>
