Commit message: Fix urdf and add world to move around

File: markhor_description/urdf/markhor.urdf.xacro (robot description, xacro)
@@ -1,70 +1,74 @@
 <?xml version="1.0"?>
-<root xmlns:xi="http://www.w3.org/2001/XInclude"
-    xmlns:xacro="http://www.ros.org/wiki/xacro">
-    <xacro:include filename="$(find markhor_description)/urdf/markhor_common.xacro" />
-    <xacro:arg name="robot_namespace" default="/" />
-    <xacro:property name="tracks_shift_x" value="0.4579783" />
-    <xacro:property name="tracks_shift_y" value="0.07620000" />
-    <xacro:property name="tracks_height" value="-0.05318760" />
-    <xacro:property name="tracks_seperation" value="${tracks_shift} * 2" />
-    <link name="base_link">
-      <visual>
-        <geometry>
-          <mesh filename="package://markhor_description/meshes/${body_mesh}.stl"/>
-        </geometry>
-        <origin xyz="0 0 0" rpy="0 0 0"/>
-      </visual>
-      <collision>
-        <geometry>
-          <mesh filename="package://markhor_description/meshes/${body_mesh}.stl"/>
-        </geometry>
-        <origin xyz="0 0 0" rpy="0 0 0"/>
-      </collision>
-      <xacro:markhor_inertial type="body"/>
-    </link>
-    <link name="base_footprint"/>
-    <joint name="base_footprint_joint" type="fixed">
-      <origin xyz="0 0 0.085" rpy="0 0 0" />
-      <parent link="base_link" />
-      <child link="base_footprint" />
-    </joint>
-    <xacro:flipper flipper_name="flipper_fl" origin_xyz="${tracks_shift_x} -${tracks_shift_y} ${tracks_height}" origin_rpy="0 0 ${-pi/2}"/>
-    <xacro:flipper flipper_name="flipper_fr" origin_xyz="${tracks_shift_x} ${tracks_shift_y} ${tracks_height}" origin_rpy="0 0 ${-pi/2}"/>
-    <xacro:flipper flipper_name="flipper_rl" origin_xyz="-${tracks_shift_x} -${tracks_shift_y} ${tracks_height}" origin_rpy="0 0 ${pi/2}"/>
-    <xacro:flipper flipper_name="flipper_rr" origin_xyz="-${tracks_shift_x} ${tracks_shift_y} ${tracks_height}" origin_rpy="0 0 ${pi/2}"/>
-    <xacro:virtual_anchor anchor_name="front_cam" parent="base_link" origin_xyz="0.35864800 0 -0.03810000" origin_rpy="0 ${pi/2} 0"/>
-    <xacro:virtual_anchor anchor_name="rear_cam" parent="base_link" origin_xyz="-0.35864800 0 -0.03810000" origin_rpy="0 ${-pi/2} 0"/>
-    <xacro:virtual_anchor anchor_name="arm_root" parent="base_link" origin_xyz="0.17394875 0 -0.12291060" origin_rpy="${pi} 0 0"/>
-    <xacro:virtual_anchor anchor_name="lidar" parent="base_link" origin_xyz="0.32034017 0 -0.1393156" origin_rpy="${pi} 0 0"/>
-    <gazebo>
-      <!-- <plugin name="gazebo_ros_control" filename="libgazebo_ros_control.so">
-        <robotNamespace>$(arg robot_namespace)</robotNamespace>
-      </plugin> -->
-      <!-- <plugin name="imu_controller" filename="libhector_gazebo_ros_imu.so">
-        <robotNamespace>$(arg robot_namespace)</robotNamespace>
-        <updateRate>50.0</updateRate>
-        <bodyName>${prefix}_link_base</bodyName>
-        <topicName>imu/data</topicName>
-        <accelDrift>0.005 0.005 0.005</accelDrift>
-        <accelGaussianNoise>0.005 0.005 0.005</accelGaussianNoise>
-        <rateDrift>0.005 0.005 0.005 </rateDrift>
-        <rateGaussianNoise>0.005 0.005 0.005 </rateGaussianNoise>
-        <headingDrift>0.005</headingDrift>
-        <headingGaussianNoise>0.005</headingGaussianNoise>
-      </plugin> -->
-      <plugin filename="libSimpleTrackedVehiclePlugin.so" name="simple_tracked_vehicle">
-        <body>base_link</body>
-        <left_track>flipper_fl</left_track>
-        <right_track>flipper_fr</right_track>
-        <left_flipper>flipper_rl</left_flipper>
-        <right_flipper>flipper_rr</right_flipper>
-        <track_mu>0.65</track_mu>
-        <track_mu2>0.85</track_mu2>
-        <tracks_separation>${tracks_seperation}</tracks_separation>
-      </plugin>
-      <plugin filename="libKeysToCmdVelPlugin.so" name="keyboard_control">
-        <publish_as_twist>true</publish_as_twist>
-        <cmd_vel_topic>~/markhor/cmd_vel_twist</cmd_vel_topic>
-      </plugin>
-    </gazebo>
-</root>
+<robot xmlns:xacro="http://www.ros.org/wiki/xacro" name="markhor">
+<xacro:include filename="$(find markhor_description)/urdf/markhor_common.xacro" />
+  <xacro:arg name="robot_namespace" default="/" />
+  <xacro:property name="tracks_shift_x" value="0.31115000" />
+  <xacro:property name="tracks_shift_y" value="0.2230283" />
+  <xacro:property name="tracks_height" value="0.05318760" />
+  <xacro:property name="tracks_seperation" value="${tracks_shift_x} * 2" />
+  <link name="base_footprint"/>
+  <link name="base_link"/>
+  <link name="base_body">
+    <visual>
+      <geometry>
+        <mesh filename="package://markhor_description/meshes/mk_link_base.stl"/>
+      </geometry>
+      <origin xyz="0 0 0" rpy="0 ${pi} 0"/>
+    </visual>
+    <collision>
+      <geometry>
+        <mesh filename="package://markhor_description/meshes/mk_link_base.stl"/>
+      </geometry>
+      <origin xyz="0 0 0" rpy="0 ${pi} 0"/>
+    </collision>
+    <xacro:markhor_inertial type="body"/>
+  </link>
+  <joint name="base_link_j" type="fixed">
+    <origin xyz="0 0 -0.085" rpy="0 0 0" />
+    <parent link="base_link" />
+    <child link="base_footprint" />
+  </joint>
+  <joint name="base_body_j" type="fixed">
+    <parent link="base_link" />
+    <child link="base_body" />
+  </joint>
+  <xacro:flipper flipper_name="flipper_fl" origin_xyz="${tracks_shift_x} ${tracks_shift_y} ${tracks_height}" origin_rpy="${pi/2} 0 ${-pi/2}"/>
+  <xacro:flipper flipper_name="flipper_fr" origin_xyz="${tracks_shift_x} -${tracks_shift_y} ${tracks_height}" origin_rpy="${pi/2} 0 ${-pi/2}"/>
+  <xacro:flipper flipper_name="flipper_rl" origin_xyz="-${tracks_shift_x} ${tracks_shift_y} ${tracks_height}" origin_rpy="${pi/2} 0 ${pi/2}"/>
+  <xacro:flipper flipper_name="flipper_rr" origin_xyz="-${tracks_shift_x} -${tracks_shift_y} ${tracks_height}" origin_rpy="${pi/2} 0 ${pi/2}"/>
+  <xacro:virtual_anchor anchor_name="front_cam" parent="base_link" origin_xyz="0.35864800 0 -0.03810000" origin_rpy="0 ${pi/2} 0"/>
+  <xacro:virtual_anchor anchor_name="rear_cam" parent="base_link" origin_xyz="-0.35864800 0 -0.03810000" origin_rpy="0 ${-pi/2} 0"/>
+  <xacro:virtual_anchor anchor_name="arm_root" parent="base_link" origin_xyz="0.17394875 0 -0.12291060" origin_rpy="${pi} 0 0"/>
+  <xacro:virtual_anchor anchor_name="lidar" parent="base_link" origin_xyz="0.32034017 0 -0.1393156" origin_rpy="${pi} 0 0"/>
+  <gazebo>
+    <!-- <plugin name="gazebo_ros_control" filename="libgazebo_ros_control.so">
+      <robotNamespace>$(arg robot_namespace)</robotNamespace>
+    </plugin> -->
+    <!-- <plugin name="imu_controller" filename="libhector_gazebo_ros_imu.so">
+      <robotNamespace>$(arg robot_namespace)</robotNamespace>
+      <updateRate>50.0</updateRate>
+      <bodyName>${prefix}_link_base</bodyName>
+      <topicName>imu/data</topicName>
+      <accelDrift>0.005 0.005 0.005</accelDrift>
+      <accelGaussianNoise>0.005 0.005 0.005</accelGaussianNoise>
+      <rateDrift>0.005 0.005 0.005 </rateDrift>
+      <rateGaussianNoise>0.005 0.005 0.005 </rateGaussianNoise>
+      <headingDrift>0.005</headingDrift>
+      <headingGaussianNoise>0.005</headingGaussianNoise>
+    </plugin> -->
+    <plugin filename="libSimpleTrackedVehiclePlugin.so" name="simple_tracked_vehicle">
+      <body>base_link</body>
+      <left_track>flipper_fl</left_track>
+      <right_track>flipper_fr</right_track>
+      <left_flipper>flipper_rl</left_flipper>
+      <right_flipper>flipper_rr</right_flipper>
+      <track_mu>0.65</track_mu>
+      <track_mu2>0.85</track_mu2>
+      <tracks_separation>${tracks_seperation}</tracks_separation>
+    </plugin>
+    <plugin filename="libKeysToCmdVelPlugin.so" name="keyboard_control">
+      <publish_as_twist>true</publish_as_twist>
+      <cmd_vel_topic>~/markhor/cmd_vel_twist</cmd_vel_topic>
+    </plugin>
+  </gazebo>
+</robot>

File: markhor_description/urdf/markhor_common.xacro (robot description, xacro)
@@ -3,6 +3,6 @@
 <root xmlns:xi="http://www.w3.org/2001/XInclude"
   xmlns:xacro="http://www.ros.org/wiki/xacro">
-  <xacro:property name="flipper_lower_limit" value="${-pi/2}"/>
-  <xacro:property name="flipper_upper_limit" value="${pi/2}" />
+  <xacro:property name="flipper_lower_limit" value="${-pi}"/>
+  <xacro:property name="flipper_upper_limit" value="0" />
   <xacro:property name="flipper_velocity_limit" value="16.75" />
   <xacro:property name="flipper_torque_limit" value="184" />
@@ -11,11 +11,10 @@
   <xacro:include filename="$(find markhor_description)/urdf/markhor_inertial.xacro" />
   <xacro:macro name="flipper" params="flipper_name origin_xyz:='0 0 0' origin_rpy:='0 0 0'">
-    <link name="${flipper_prefix}">
+    <link name="${flipper_name}">
       <visual>
         <geometry>
           <mesh filename="package://markhor_description/meshes/mk_flip.stl"/>
         </geometry>
-        <origin xyz="${origin_xyz}" rpy="${origin_rpy}"/>
-        <material name="${link_material}"/>
+        <origin xyz="0 0 0" rpy="0 0 0"/>
       </visual>
       <collision>
@@ -23,5 +22,5 @@
           <mesh filename="package://markhor_description/meshes/mk_flip.stl"/>
         </geometry>
-        <origin xyz="${origin_xyz}" rpy="${origin_rpy}"/>
+        <origin xyz="0 0 0" rpy="0 0 0"/>
         <surface>
           <friction>
@@ -40,11 +39,11 @@
       <xacro:markhor_inertial type="flipper"/>
     </link>
-    <link name="${flipper_prefix}_motor">
+    <link name="${flipper_name}_motor">
       <xacro:markhor_inertial type="motor"/>
     </link>
-    <joint name="${flipper_prefix}_j" type="revolute">
+    <joint name="${flipper_name}_j" type="revolute">
 			<parent link="base_link"/>
-			<child link="${flipper_prefix}"/>
-			<axis xyz="0 1 0" rpy="0 0 0" />
+			<child link="${flipper_name}"/>
+			<axis xyz="1 0 0" rpy="0 0 0" />
       <origin xyz="${origin_xyz}" rpy="${origin_rpy}"/>
       <limit effort="${flipper_torque_limit}" velocity="${flipper_velocity_limit}" lower="${flipper_lower_limit}" upper="${flipper_upper_limit}"/>
@@ -60,25 +59,25 @@
         </ode>
       </physics>
-      <transmission name="${flipper_prefix}_trans">
+      <transmission name="${flipper_name}_trans">
         <type>transmission_interface/SimpleTransmission</type>
-        <joint name="${flipper_prefix}_j">
+        <joint name="${flipper_name}_j">
           <hardwareInterface>hardware_interface/EffortJointInterface</hardwareInterface>
         </joint>
-        <actuator name="${flipper_prefix}_actuator">
+        <actuator name="${flipper_name}_actuator">
           <mechanicalReduction>1</mechanicalReduction>
         </actuator>
       </transmission>
 		</joint>
-    <joint name="${flipper_prefix}_motor_j" type="continuous">
-			<parent link="${flipper_prefix}"/>
-			<child link="${flipper_prefix}_motor"/>
-			<axis xyz="0 1 0" rpy="0 0 0" />
+    <joint name="${flipper_name}_motor_j" type="continuous">
+			<parent link="${flipper_name}"/>
+			<child link="${flipper_name}_motor"/>
+			<axis xyz="1 0 0" rpy="0 0 0" />
       <limit effort="${track_torque_limit}" velocity="${track_velocity_limit}"/>
-      <transmission name="${flipper_prefix}_track_trans" type="SimpleTransmission">
+      <transmission name="${flipper_name}_track_trans" type="SimpleTransmission">
         <type>transmission_interface/SimpleTransmission</type>
-        <joint name="${flipper_prefix}_motor_j">
+        <joint name="${flipper_name}_motor_j">
           <hardwareInterface>hardware_interface/VelocityJointInterface</hardwareInterface>
         </joint>
-        <actuator name="${flipper_prefix}_track_motor">
+        <actuator name="${flipper_name}_track_motor">
           <mechanicalReduction>1</mechanicalReduction>
         </actuator>

Commit message: Add ros_control for the flipper

File: markhor_description/urdf/markhor.urdf.xacro (robot description, xacro)
@@ -2,5 +2,5 @@
 <robot xmlns:xacro="http://www.ros.org/wiki/xacro" name="markhor">
 <xacro:include filename="$(find markhor_description)/urdf/markhor_common.xacro" />
-  <xacro:arg name="robot_namespace" default="/" />
+  <xacro:arg name="robot_namespace" default="/markhor" />
   <xacro:property name="tracks_shift_x" value="0.31115000" />
   <xacro:property name="tracks_shift_y" value="0.2230283" />
@@ -42,7 +42,7 @@
   <xacro:virtual_anchor anchor_name="lidar" parent="base_link" origin_xyz="0.32034017 0 -0.1393156" origin_rpy="${pi} 0 0"/>
   <gazebo>
-    <!-- <plugin name="gazebo_ros_control" filename="libgazebo_ros_control.so">
+    <plugin name="gazebo_ros_control" filename="libgazebo_ros_control.so">
       <robotNamespace>$(arg robot_namespace)</robotNamespace>
-    </plugin> -->
+    </plugin>
     <!-- <plugin name="imu_controller" filename="libhector_gazebo_ros_imu.so">
       <robotNamespace>$(arg robot_namespace)</robotNamespace>

File: markhor_description/urdf/markhor_common.xacro (robot description, xacro)
@@ -28,5 +28,4 @@
               <mu>0.65</mu>
               <mu2>0.85</mu2>
-              <fdir1>0 1 0</fdir1>
             </ode>
           </friction>
@@ -48,24 +47,8 @@
       <origin xyz="${origin_xyz}" rpy="${origin_rpy}"/>
       <limit effort="${flipper_torque_limit}" velocity="${flipper_velocity_limit}" lower="${flipper_lower_limit}" upper="${flipper_upper_limit}"/>
-      <dynamics damping="0.0" friction="0.0"/>
       <physics>
         <ode>
-          <implicit_spring_damper>1</implicit_spring_damper>
-          <cfm_damping>1</cfm_damping>
-          <limit>
-            <cfm>0</cfm>
-            <erp>0.2</erp>
-          </limit>
         </ode>
       </physics>
-      <transmission name="${flipper_name}_trans">
-        <type>transmission_interface/SimpleTransmission</type>
-        <joint name="${flipper_name}_j">
-          <hardwareInterface>hardware_interface/EffortJointInterface</hardwareInterface>
-        </joint>
-        <actuator name="${flipper_name}_actuator">
-          <mechanicalReduction>1</mechanicalReduction>
-        </actuator>
-      </transmission>
 		</joint>
     <joint name="${flipper_name}_motor_j" type="continuous">
@@ -74,14 +57,23 @@
 			<axis xyz="1 0 0" rpy="0 0 0" />
       <limit effort="${track_torque_limit}" velocity="${track_velocity_limit}"/>
-      <transmission name="${flipper_name}_track_trans" type="SimpleTransmission">
-        <type>transmission_interface/SimpleTransmission</type>
-        <joint name="${flipper_name}_motor_j">
-          <hardwareInterface>hardware_interface/VelocityJointInterface</hardwareInterface>
-        </joint>
-        <actuator name="${flipper_name}_track_motor">
-          <mechanicalReduction>1</mechanicalReduction>
-        </actuator>
-      </transmission>
 		</joint>
+    <transmission name="${flipper_name}_trans">
+      <type>transmission_interface/SimpleTransmission</type>
+      <joint name="${flipper_name}_j">
+        <hardwareInterface>hardware_interface/EffortJointInterface</hardwareInterface>
+      </joint>
+      <actuator name="${flipper_name}_actuator">
+        <mechanicalReduction>1</mechanicalReduction>
+      </actuator>
+    </transmission>
+    <transmission name="${flipper_name}_track_trans" type="SimpleTransmission">
+      <type>transmission_interface/SimpleTransmission</type>
+      <joint name="${flipper_name}_motor_j">
+        <hardwareInterface>hardware_interface/VelocityJointInterface</hardwareInterface>
+      </joint>
+      <actuator name="${flipper_name}_track_motor">
+        <mechanicalReduction>1</mechanicalReduction>
+      </actuator>
+    </transmission>
   </xacro:macro>
   <xacro:macro name="virtual_anchor" params="anchor_name parent origin_xyz origin_rpy">

Commit message: Fix tracks simulation

File: markhor_description/urdf/markhor.urdf.xacro (robot description, xacro)
@@ -6,5 +6,5 @@
   <xacro:property name="tracks_shift_y" value="0.2230283" />
   <xacro:property name="tracks_height" value="0.05318760" />
-  <xacro:property name="tracks_seperation" value="${tracks_shift_x} * 2" />
+  <xacro:property name="tracks_seperation" value="${tracks_shift_y} * 2" />
   <link name="base_footprint"/>
   <link name="base_link"/>

Commit message: Add lidar and camera sensors

File: markhor_description/urdf/markhor.urdf.xacro (robot description, xacro)
@@ -1,6 +1,7 @@
 <?xml version="1.0"?>
 <robot xmlns:xacro="http://www.ros.org/wiki/xacro" name="markhor">
+<xacro:include filename="$(find sick_tim)/urdf/sick_tim.urdf.xacro"/>
 <xacro:include filename="$(find markhor_description)/urdf/markhor_common.xacro" />
-  <xacro:arg name="robot_namespace" default="/markhor" />
+  <xacro:arg name="robot_namespace" default="markhor" />
   <xacro:property name="tracks_shift_x" value="0.31115000" />
   <xacro:property name="tracks_shift_y" value="0.2230283" />
@@ -37,11 +38,12 @@
   <xacro:flipper flipper_name="flipper_rl" origin_xyz="-${tracks_shift_x} ${tracks_shift_y} ${tracks_height}" origin_rpy="${pi/2} 0 ${pi/2}"/>
   <xacro:flipper flipper_name="flipper_rr" origin_xyz="-${tracks_shift_x} -${tracks_shift_y} ${tracks_height}" origin_rpy="${pi/2} 0 ${pi/2}"/>
-  <xacro:virtual_anchor anchor_name="front_cam" parent="base_link" origin_xyz="0.35864800 0 -0.03810000" origin_rpy="0 ${pi/2} 0"/>
-  <xacro:virtual_anchor anchor_name="rear_cam" parent="base_link" origin_xyz="-0.35864800 0 -0.03810000" origin_rpy="0 ${-pi/2} 0"/>
-  <xacro:virtual_anchor anchor_name="arm_root" parent="base_link" origin_xyz="0.17394875 0 -0.12291060" origin_rpy="${pi} 0 0"/>
-  <xacro:virtual_anchor anchor_name="lidar" parent="base_link" origin_xyz="0.32034017 0 -0.1393156" origin_rpy="${pi} 0 0"/>
+  <xacro:camera_link link_name="front_cam" camera_name="$(arg robot_namespace)/front_cam" frame_name="front_cam" parent="base_link" origin_xyz="0.35864800 0 0.03810000" origin_rpy="0 0 0"/>
+  <xacro:camera_link link_name="rear_cam" camera_name="$(arg robot_namespace)/rear_cam" frame_name="rear_cam" parent="base_link" origin_xyz="-0.35864800 0 0.03810000" origin_rpy="0 0 ${pi}"/>
+  <xacro:virtual_anchor anchor_name="arm_root" parent="base_link" origin_xyz="0.17394875 0 0.12291060" origin_rpy="0 0 0"/>
+  <xacro:sick_tim551 name="laser" ros_topic="scan"/>
+  <xacro:virtual_joint name="laser_mount_link" parent="base_link" origin_xyz="0.32034017 0 0.1393156" origin_rpy="0 0 0"/>
   <gazebo>
     <plugin name="gazebo_ros_control" filename="libgazebo_ros_control.so">
-      <robotNamespace>$(arg robot_namespace)</robotNamespace>
+      <robotNamespace>/$(arg robot_namespace)</robotNamespace>
     </plugin>
     <!-- <plugin name="imu_controller" filename="libhector_gazebo_ros_imu.so">

File: markhor_description/urdf/markhor_common.xacro (robot description, xacro)
@@ -39,5 +39,5 @@
     </link>
     <link name="${flipper_name}_motor">
-      <xacro:markhor_inertial type="motor"/>
+      <xacro:markhor_inertial type="virtual"/>
     </link>
     <joint name="${flipper_name}_j" type="revolute">
@@ -75,5 +75,7 @@
   </xacro:macro>
   <xacro:macro name="virtual_anchor" params="anchor_name parent origin_xyz origin_rpy">
-    <link name="${anchor_name}"/>
+    <link name="${anchor_name}">
+      <xacro:markhor_inertial type="virtual"/>
+    </link>
     <joint name="${anchor_name}_j" type="fixed">
       <parent link="${parent}"/>
@@ -82,3 +84,61 @@
     </joint>
   </xacro:macro>
+  <xacro:macro name="virtual_joint" params="name parent origin_xyz origin_rpy">
+    <joint name="${name}_j" type="fixed">
+      <parent link="${parent}"/>
+      <child link="${name}"/>
+      <origin xyz="${origin_xyz}" rpy="${origin_rpy}"/>
+    </joint>
+  </xacro:macro>
+  <xacro:macro name="camera_link" params="link_name camera_name frame_name parent origin_xyz origin_rpy">
+    <link name="${link_name}">
+      <xacro:markhor_inertial type="virtual"/>
+    </link>
+    <joint name="${link_name}_j" type="fixed">
+      <parent link="${parent}"/>
+      <child link="${link_name}"/>
+      <origin xyz="${origin_xyz}" rpy="${origin_rpy}"/>
+    </joint>
+    <gazebo reference="${link_name}">
+      <sensor name="${link_name}_camera" type="depth">
+        <update_rate>60</update_rate>
+        <camera>
+          <horizontal_fov>1.047198</horizontal_fov>
+          <image>
+            <width>640</width>
+            <height>400</height>
+            <format>R8G8B8</format>
+          </image>
+          <clip>
+            <near>0.25</near>
+            <far>1.5</far>
+          </clip>
+        </camera>
+        <plugin name="${link_name}_controller" filename="libgazebo_ros_openni_kinect.so">
+          <baseline>0.2</baseline>
+          <alwaysOn>true</alwaysOn>
+          <updateRate>1.0</updateRate>
+          <cameraName>${camera_name}_ir</cameraName>
+          <imageTopicName>/${camera_name}/color/image_raw</imageTopicName>
+          <cameraInfoTopicName>/${camera_name}/color/camera_info</cameraInfoTopicName>
+          <depthImageTopicName>/${camera_name}/depth/image_raw</depthImageTopicName>
+          <depthImageInfoTopicName>/${camera_name}/depth/camera_info</depthImageInfoTopicName>
+          <pointCloudTopicName>/${camera_name}/depth/points</pointCloudTopicName>
+          <frameName>${frame_name}</frameName>
+          <pointCloudCutoff>0.5</pointCloudCutoff>
+          <pointCloudCutoffMax>3.0</pointCloudCutoffMax>
+          <distortionK1>0.00000001</distortionK1>
+          <distortionK2>0.00000001</distortionK2>
+          <distortionK3>0.00000001</distortionK3>
+          <distortionT1>0.00000001</distortionT1>
+          <distortionT2>0.00000001</distortionT2>
+          <CxPrime>0</CxPrime>
+          <Cx>0</Cx>
+          <Cy>0</Cy>
+          <focalLength>0</focalLength>
+          <hackBaseline>0</hackBaseline>
+        </plugin>
+      </sensor>
+    </gazebo>
+  </xacro:macro>
 </root>

File: markhor_description/urdf/markhor_inertial.xacro (robot description, xacro)
@@ -25,8 +25,8 @@
             </inertial>
         </xacro:if>
-        <xacro:if value="${type == 'motor'}">
+        <xacro:if value="${type == 'virtual'}">
             <inertial>
                 <mass value="0.0001"/>
-                <origin xyz="0 0.116 0" rpy="0 0 0"/>
+                <origin xyz="0 0 0" rpy="0 0 0"/>
                 <inertia
                     ixx="0.001" ixy="0" ixz="0"
