Commit message: Convert tabs to space and set the default to 4 instead of 2

File: markhor_description/urdf/markhor.urdf.xacro (robot description, xacro)
@@ -1,51 +1,51 @@
 <?xml version="1.0"?>
 <robot xmlns:xacro="http://www.ros.org/wiki/xacro" name="markhor">
-  <xacro:include filename="$(find sick_tim)/urdf/sick_tim.urdf.xacro" />
-  <xacro:include filename="$(find markhor_description)/urdf/markhor_common.xacro" />
-  <xacro:arg name="robot_namespace" default="markhor" />
-  <xacro:property name="tracks_shift_x" value="0.31115000" />
-  <xacro:property name="tracks_shift_y" value="0.2230283" />
-  <xacro:property name="tracks_height" value="0.05318760" />
-  <xacro:property name="tracks_seperation" value="${tracks_shift_y} * 2" />
-  <link name="base_footprint" />
-  <link name="base_link" />
-  <link name="base_body">
-    <visual>
-      <geometry>
-        <mesh filename="package://markhor_description/meshes/mk_link_base.stl" />
-      </geometry>
-      <origin xyz="0 0 0" rpy="0 ${pi} 0" />
-    </visual>
-    <collision>
-      <geometry>
-        <mesh filename="package://markhor_description/meshes/mk_link_base.stl" />
-      </geometry>
-      <origin xyz="0 0 0" rpy="0 ${pi} 0" />
-    </collision>
-    <xacro:markhor_inertial type="body" />
-  </link>
-  <joint name="base_link_j" type="fixed">
-    <origin xyz="0 0 -0.085" rpy="0 0 0" />
-    <parent link="base_link" />
-    <child link="base_footprint" />
-  </joint>
-  <joint name="base_body_j" type="fixed">
-    <parent link="base_link" />
-    <child link="base_body" />
-  </joint>
-  <xacro:flipper flipper_name="flipper_fl" origin_xyz="${tracks_shift_x} ${tracks_shift_y} ${tracks_height}" origin_rpy="${pi/2} 0 ${-pi/2}" />
-  <xacro:flipper flipper_name="flipper_fr" origin_xyz="${tracks_shift_x} -${tracks_shift_y} ${tracks_height}" origin_rpy="${pi/2} 0 ${-pi/2}" />
-  <xacro:flipper flipper_name="flipper_rl" origin_xyz="-${tracks_shift_x} ${tracks_shift_y} ${tracks_height}" origin_rpy="${pi/2} 0 ${pi/2}" />
-  <xacro:flipper flipper_name="flipper_rr" origin_xyz="-${tracks_shift_x} -${tracks_shift_y} ${tracks_height}" origin_rpy="${pi/2} 0 ${pi/2}" />
-  <xacro:camera_link link_name="front_cam" camera_name="$(arg robot_namespace)/front_cam" frame_name="front_cam" parent="base_link" origin_xyz="0.35864800 0 0.03810000" origin_rpy="0 0 0" />
-  <xacro:camera_link link_name="rear_cam" camera_name="$(arg robot_namespace)/rear_cam" frame_name="rear_cam" parent="base_link" origin_xyz="-0.35864800 0 0.03810000" origin_rpy="0 0 ${pi}" />
-  <xacro:virtual_anchor anchor_name="arm_root" parent="base_link" origin_xyz="0.17394875 0 0.12291060" origin_rpy="0 0 0" />
-  <xacro:sick_tim551 name="laser" ros_topic="scan" />
-  <xacro:virtual_joint name="laser_mount_link" parent="base_link" origin_xyz="0.32034017 0 0.1393156" origin_rpy="0 0 0" />
-  <gazebo>
-    <plugin name="gazebo_ros_control" filename="libgazebo_ros_control.so">
-      <robotNamespace>/$(arg robot_namespace)</robotNamespace>
-    </plugin>
-    <!-- <plugin name="imu_controller" filename="libhector_gazebo_ros_imu.so">
+    <xacro:include filename="$(find sick_tim)/urdf/sick_tim.urdf.xacro" />
+    <xacro:include filename="$(find markhor_description)/urdf/markhor_common.xacro" />
+    <xacro:arg name="robot_namespace" default="markhor" />
+    <xacro:property name="tracks_shift_x" value="0.31115000" />
+    <xacro:property name="tracks_shift_y" value="0.2230283" />
+    <xacro:property name="tracks_height" value="0.05318760" />
+    <xacro:property name="tracks_seperation" value="${tracks_shift_y} * 2" />
+    <link name="base_footprint" />
+    <link name="base_link" />
+    <link name="base_body">
+        <visual>
+            <geometry>
+                <mesh filename="package://markhor_description/meshes/mk_link_base.stl" />
+            </geometry>
+            <origin xyz="0 0 0" rpy="0 ${pi} 0" />
+        </visual>
+        <collision>
+            <geometry>
+                <mesh filename="package://markhor_description/meshes/mk_link_base.stl" />
+            </geometry>
+            <origin xyz="0 0 0" rpy="0 ${pi} 0" />
+        </collision>
+        <xacro:markhor_inertial type="body" />
+    </link>
+    <joint name="base_link_j" type="fixed">
+        <origin xyz="0 0 -0.085" rpy="0 0 0" />
+        <parent link="base_link" />
+        <child link="base_footprint" />
+    </joint>
+    <joint name="base_body_j" type="fixed">
+        <parent link="base_link" />
+        <child link="base_body" />
+    </joint>
+    <xacro:flipper flipper_name="flipper_fl" origin_xyz="${tracks_shift_x} ${tracks_shift_y} ${tracks_height}" origin_rpy="${pi/2} 0 ${-pi/2}" />
+    <xacro:flipper flipper_name="flipper_fr" origin_xyz="${tracks_shift_x} -${tracks_shift_y} ${tracks_height}" origin_rpy="${pi/2} 0 ${-pi/2}" />
+    <xacro:flipper flipper_name="flipper_rl" origin_xyz="-${tracks_shift_x} ${tracks_shift_y} ${tracks_height}" origin_rpy="${pi/2} 0 ${pi/2}" />
+    <xacro:flipper flipper_name="flipper_rr" origin_xyz="-${tracks_shift_x} -${tracks_shift_y} ${tracks_height}" origin_rpy="${pi/2} 0 ${pi/2}" />
+    <xacro:camera_link link_name="front_cam" camera_name="$(arg robot_namespace)/front_cam" frame_name="front_cam" parent="base_link" origin_xyz="0.35864800 0 0.03810000" origin_rpy="0 0 0" />
+    <xacro:camera_link link_name="rear_cam" camera_name="$(arg robot_namespace)/rear_cam" frame_name="rear_cam" parent="base_link" origin_xyz="-0.35864800 0 0.03810000" origin_rpy="0 0 ${pi}" />
+    <xacro:virtual_anchor anchor_name="arm_root" parent="base_link" origin_xyz="0.17394875 0 0.12291060" origin_rpy="0 0 0" />
+    <xacro:sick_tim551 name="laser" ros_topic="scan" />
+    <xacro:virtual_joint name="laser_mount_link" parent="base_link" origin_xyz="0.32034017 0 0.1393156" origin_rpy="0 0 0" />
+    <gazebo>
+        <plugin name="gazebo_ros_control" filename="libgazebo_ros_control.so">
+            <robotNamespace>/$(arg robot_namespace)</robotNamespace>
+        </plugin>
+        <!-- <plugin name="imu_controller" filename="libhector_gazebo_ros_imu.so">
       <robotNamespace>$(arg robot_namespace)</robotNamespace>
       <updateRate>50.0</updateRate>
@@ -59,18 +59,18 @@
       <headingGaussianNoise>0.005</headingGaussianNoise>
     </plugin> -->
-    <plugin filename="libSimpleTrackedVehiclePlugin.so" name="simple_tracked_vehicle">
-      <body>base_link</body>
-      <left_track>flipper_fl</left_track>
-      <right_track>flipper_fr</right_track>
-      <left_flipper>flipper_rl</left_flipper>
-      <right_flipper>flipper_rr</right_flipper>
-      <track_mu>0.65</track_mu>
-      <track_mu2>0.85</track_mu2>
-      <tracks_separation>${tracks_seperation}</tracks_separation>
-    </plugin>
-    <plugin filename="libKeysToCmdVelPlugin.so" name="keyboard_control">
-      <publish_as_twist>true</publish_as_twist>
-      <cmd_vel_topic>~/markhor/cmd_vel_twist</cmd_vel_topic>
-    </plugin>
-  </gazebo>
+        <plugin filename="libSimpleTrackedVehiclePlugin.so" name="simple_tracked_vehicle">
+            <body>base_link</body>
+            <left_track>flipper_fl</left_track>
+            <right_track>flipper_fr</right_track>
+            <left_flipper>flipper_rl</left_flipper>
+            <right_flipper>flipper_rr</right_flipper>
+            <track_mu>0.65</track_mu>
+            <track_mu2>0.85</track_mu2>
+            <tracks_separation>${tracks_seperation}</tracks_separation>
+        </plugin>
+        <!-- <plugin filename="libKeysToCmdVelPlugin.so" name="keyboard_control">
+            <publish_as_twist>true</publish_as_twist>
+            <cmd_vel_topic>~/markhor/cmd_vel_twist</cmd_vel_topic>
+        </plugin> -->
+    </gazebo>
 </robot>

File: markhor_description/urdf/markhor_common.xacro (robot description, xacro)
@@ -2,143 +2,143 @@
 <!-- Adapted from the kinova-ros pkg for use by Club Capra on the markhor robotic platform -->
 <root xmlns:xi="http://www.w3.org/2001/XInclude"
-  xmlns:xacro="http://www.ros.org/wiki/xacro">
-  <xacro:property name="flipper_lower_limit" value="${-pi}"/>
-  <xacro:property name="flipper_upper_limit" value="0" />
-  <xacro:property name="flipper_velocity_limit" value="16.75" />
-  <xacro:property name="flipper_torque_limit" value="184" />
-  <xacro:property name="track_velocity_limit" value="5.34" />
-  <xacro:property name="track_torque_limit" value="94.5" />
-  <xacro:include filename="$(find markhor_description)/urdf/markhor_inertial.xacro" />
-  <xacro:macro name="flipper" params="flipper_name origin_xyz:='0 0 0' origin_rpy:='0 0 0'">
-    <link name="${flipper_name}">
-      <visual>
-        <geometry>
-          <mesh filename="package://markhor_description/meshes/mk_flip.stl"/>
-        </geometry>
-        <origin xyz="0 0 0" rpy="0 0 0"/>
-      </visual>
-      <collision>
-        <geometry>
-          <mesh filename="package://markhor_description/meshes/mk_flip.stl"/>
-        </geometry>
-        <origin xyz="0 0 0" rpy="0 0 0"/>
-        <surface>
-          <friction>
-            <ode>
-              <mu>0.65</mu>
-              <mu2>0.85</mu2>
-            </ode>
-          </friction>
-          <contact>
-            <ode/>
-          </contact>
-        </surface>
-      </collision>
-      <max_contacts>20</max_contacts>
-      <xacro:markhor_inertial type="flipper"/>
-    </link>
-    <link name="${flipper_name}_motor">
-      <xacro:markhor_inertial type="virtual"/>
-    </link>
-    <joint name="${flipper_name}_j" type="revolute">
-			<parent link="base_link"/>
-			<child link="${flipper_name}"/>
-			<axis xyz="1 0 0" rpy="0 0 0" />
-      <origin xyz="${origin_xyz}" rpy="${origin_rpy}"/>
-      <limit effort="${flipper_torque_limit}" velocity="${flipper_velocity_limit}" lower="${flipper_lower_limit}" upper="${flipper_upper_limit}"/>
-      <dynamics damping="150"/>
-    </joint>
-    <joint name="${flipper_name}_motor_j" type="continuous">
-			<parent link="${flipper_name}"/>
-			<child link="${flipper_name}_motor"/>
-			<axis xyz="1 0 0" rpy="0 0 0" />
-      <limit effort="${track_torque_limit}" velocity="${track_velocity_limit}"/>
-		</joint>
-    <transmission name="${flipper_name}_trans">
-      <type>transmission_interface/SimpleTransmission</type>
-      <joint name="${flipper_name}_j">
-        <hardwareInterface>hardware_interface/EffortJointInterface</hardwareInterface>
-      </joint>
-      <actuator name="${flipper_name}_actuator">
-        <mechanicalReduction>1</mechanicalReduction>
-      </actuator>
-    </transmission>
-    <transmission name="${flipper_name}_track_trans" type="SimpleTransmission">
-      <type>transmission_interface/SimpleTransmission</type>
-      <joint name="${flipper_name}_motor_j">
-        <hardwareInterface>hardware_interface/VelocityJointInterface</hardwareInterface>
-      </joint>
-      <actuator name="${flipper_name}_track_motor">
-        <mechanicalReduction>1</mechanicalReduction>
-      </actuator>
-    </transmission>
-  </xacro:macro>
-  <xacro:macro name="virtual_anchor" params="anchor_name parent origin_xyz origin_rpy">
-    <link name="${anchor_name}">
-      <xacro:markhor_inertial type="virtual"/>
-    </link>
-    <joint name="${anchor_name}_j" type="fixed">
-      <parent link="${parent}"/>
-      <child link="${anchor_name}"/>
-      <origin xyz="${origin_xyz}" rpy="${origin_rpy}"/>
-    </joint>
-  </xacro:macro>
-  <xacro:macro name="virtual_joint" params="name parent origin_xyz origin_rpy">
-    <joint name="${name}_j" type="fixed">
-      <parent link="${parent}"/>
-      <child link="${name}"/>
-      <origin xyz="${origin_xyz}" rpy="${origin_rpy}"/>
-    </joint>
-  </xacro:macro>
-  <xacro:macro name="camera_link" params="link_name camera_name frame_name parent origin_xyz origin_rpy">
-    <link name="${link_name}">
-      <xacro:markhor_inertial type="virtual"/>
-    </link>
-    <joint name="${link_name}_j" type="fixed">
-      <parent link="${parent}"/>
-      <child link="${link_name}"/>
-      <origin xyz="${origin_xyz}" rpy="${origin_rpy}"/>
-    </joint>
-    <gazebo reference="${link_name}">
-      <sensor name="${link_name}_camera" type="depth">
-        <update_rate>60</update_rate>
-        <camera>
-          <horizontal_fov>1.047198</horizontal_fov>
-          <image>
-            <width>640</width>
-            <height>400</height>
-            <format>R8G8B8</format>
-          </image>
-          <clip>
-            <near>0.25</near>
-            <far>1.5</far>
-          </clip>
-        </camera>
-        <plugin name="${link_name}_controller" filename="libgazebo_ros_openni_kinect.so">
-          <baseline>0.2</baseline>
-          <alwaysOn>true</alwaysOn>
-          <updateRate>1.0</updateRate>
-          <cameraName>${camera_name}_ir</cameraName>
-          <imageTopicName>/${camera_name}/color/image_raw</imageTopicName>
-          <cameraInfoTopicName>/${camera_name}/color/camera_info</cameraInfoTopicName>
-          <depthImageTopicName>/${camera_name}/depth/image_raw</depthImageTopicName>
-          <depthImageInfoTopicName>/${camera_name}/depth/camera_info</depthImageInfoTopicName>
-          <pointCloudTopicName>/${camera_name}/depth/points</pointCloudTopicName>
-          <frameName>${frame_name}</frameName>
-          <pointCloudCutoff>0.5</pointCloudCutoff>
-          <pointCloudCutoffMax>3.0</pointCloudCutoffMax>
-          <distortionK1>0.00000001</distortionK1>
-          <distortionK2>0.00000001</distortionK2>
-          <distortionK3>0.00000001</distortionK3>
-          <distortionT1>0.00000001</distortionT1>
-          <distortionT2>0.00000001</distortionT2>
-          <CxPrime>0</CxPrime>
-          <Cx>0</Cx>
-          <Cy>0</Cy>
-          <focalLength>0</focalLength>
-          <hackBaseline>0</hackBaseline>
-        </plugin>
-      </sensor>
-    </gazebo>
-  </xacro:macro>
+    xmlns:xacro="http://www.ros.org/wiki/xacro">
+    <xacro:property name="flipper_lower_limit" value="${-pi}"/>
+    <xacro:property name="flipper_upper_limit" value="0" />
+    <xacro:property name="flipper_velocity_limit" value="16.75" />
+    <xacro:property name="flipper_torque_limit" value="184" />
+    <xacro:property name="track_velocity_limit" value="5.34" />
+    <xacro:property name="track_torque_limit" value="94.5" />
+    <xacro:include filename="$(find markhor_description)/urdf/markhor_inertial.xacro" />
+    <xacro:macro name="flipper" params="flipper_name origin_xyz:='0 0 0' origin_rpy:='0 0 0'">
+        <link name="${flipper_name}">
+            <visual>
+                <geometry>
+                    <mesh filename="package://markhor_description/meshes/mk_flip.stl"/>
+                </geometry>
+                <origin xyz="0 0 0" rpy="0 0 0"/>
+            </visual>
+            <collision>
+                <geometry>
+                    <mesh filename="package://markhor_description/meshes/mk_flip.stl"/>
+                </geometry>
+                <origin xyz="0 0 0" rpy="0 0 0"/>
+                <surface>
+                    <friction>
+                        <ode>
+                            <mu>0.65</mu>
+                            <mu2>0.85</mu2>
+                        </ode>
+                    </friction>
+                    <contact>
+                        <ode/>
+                    </contact>
+                </surface>
+            </collision>
+            <max_contacts>20</max_contacts>
+            <xacro:markhor_inertial type="flipper"/>
+        </link>
+        <link name="${flipper_name}_motor">
+            <xacro:markhor_inertial type="virtual"/>
+        </link>
+        <joint name="${flipper_name}_j" type="revolute">
+            <parent link="base_link"/>
+            <child link="${flipper_name}"/>
+            <axis xyz="1 0 0" rpy="0 0 0" />
+            <origin xyz="${origin_xyz}" rpy="${origin_rpy}"/>
+            <limit effort="${flipper_torque_limit}" velocity="${flipper_velocity_limit}" lower="${flipper_lower_limit}" upper="${flipper_upper_limit}"/>
+            <dynamics damping="150"/>
+        </joint>
+        <joint name="${flipper_name}_motor_j" type="continuous">
+            <parent link="${flipper_name}"/>
+            <child link="${flipper_name}_motor"/>
+            <axis xyz="1 0 0" rpy="0 0 0" />
+            <limit effort="${track_torque_limit}" velocity="${track_velocity_limit}"/>
+        </joint>
+        <transmission name="${flipper_name}_trans">
+            <type>transmission_interface/SimpleTransmission</type>
+            <joint name="${flipper_name}_j">
+                <hardwareInterface>hardware_interface/EffortJointInterface</hardwareInterface>
+            </joint>
+            <actuator name="${flipper_name}_actuator">
+                <mechanicalReduction>1</mechanicalReduction>
+            </actuator>
+        </transmission>
+        <transmission name="${flipper_name}_track_trans" type="SimpleTransmission">
+            <type>transmission_interface/SimpleTransmission</type>
+            <joint name="${flipper_name}_motor_j">
+                <hardwareInterface>hardware_interface/VelocityJointInterface</hardwareInterface>
+            </joint>
+            <actuator name="${flipper_name}_track_motor">
+                <mechanicalReduction>1</mechanicalReduction>
+            </actuator>
+        </transmission>
+    </xacro:macro>
+    <xacro:macro name="virtual_anchor" params="anchor_name parent origin_xyz origin_rpy">
+        <link name="${anchor_name}">
+            <xacro:markhor_inertial type="virtual"/>
+        </link>
+        <joint name="${anchor_name}_j" type="fixed">
+            <parent link="${parent}"/>
+            <child link="${anchor_name}"/>
+            <origin xyz="${origin_xyz}" rpy="${origin_rpy}"/>
+        </joint>
+    </xacro:macro>
+    <xacro:macro name="virtual_joint" params="name parent origin_xyz origin_rpy">
+        <joint name="${name}_j" type="fixed">
+            <parent link="${parent}"/>
+            <child link="${name}"/>
+            <origin xyz="${origin_xyz}" rpy="${origin_rpy}"/>
+        </joint>
+    </xacro:macro>
+    <xacro:macro name="camera_link" params="link_name camera_name frame_name parent origin_xyz origin_rpy">
+        <link name="${link_name}">
+            <xacro:markhor_inertial type="virtual"/>
+        </link>
+        <joint name="${link_name}_j" type="fixed">
+            <parent link="${parent}"/>
+            <child link="${link_name}"/>
+            <origin xyz="${origin_xyz}" rpy="${origin_rpy}"/>
+        </joint>
+        <gazebo reference="${link_name}">
+            <sensor name="${link_name}_camera" type="depth">
+                <update_rate>60</update_rate>
+                <camera>
+                    <horizontal_fov>1.047198</horizontal_fov>
+                    <image>
+                        <width>640</width>
+                        <height>400</height>
+                        <format>R8G8B8</format>
+                    </image>
+                    <clip>
+                        <near>0.25</near>
+                        <far>1.5</far>
+                    </clip>
+                </camera>
+                <plugin name="${link_name}_controller" filename="libgazebo_ros_openni_kinect.so">
+                    <baseline>0.2</baseline>
+                    <alwaysOn>true</alwaysOn>
+                    <updateRate>1.0</updateRate>
+                    <cameraName>${camera_name}_ir</cameraName>
+                    <imageTopicName>/${camera_name}/color/image_raw</imageTopicName>
+                    <cameraInfoTopicName>/${camera_name}/color/camera_info</cameraInfoTopicName>
+                    <depthImageTopicName>/${camera_name}/depth/image_raw</depthImageTopicName>
+                    <depthImageInfoTopicName>/${camera_name}/depth/camera_info</depthImageInfoTopicName>
+                    <pointCloudTopicName>/${camera_name}/depth/points</pointCloudTopicName>
+                    <frameName>${frame_name}</frameName>
+                    <pointCloudCutoff>0.5</pointCloudCutoff>
+                    <pointCloudCutoffMax>3.0</pointCloudCutoffMax>
+                    <distortionK1>0.00000001</distortionK1>
+                    <distortionK2>0.00000001</distortionK2>
+                    <distortionK3>0.00000001</distortionK3>
+                    <distortionT1>0.00000001</distortionT1>
+                    <distortionT2>0.00000001</distortionT2>
+                    <CxPrime>0</CxPrime>
+                    <Cx>0</Cx>
+                    <Cy>0</Cy>
+                    <focalLength>0</focalLength>
+                    <hackBaseline>0</hackBaseline>
+                </plugin>
+            </sensor>
+        </gazebo>
+    </xacro:macro>
 </root>
