Commit message: Fixed Broken PID for flippers, Integrated Tracks Interface

File: markhor_description/urdf/markhor.urdf.xacro (robot description, xacro)
@@ -43,4 +43,22 @@
     <xacro:sick_tim551 name="laser" ros_topic="scan" />
     <xacro:virtual_joint name="laser_mount_link" parent="base_link" origin_xyz="0.32034017 0 0.1393156" origin_rpy="0 0 0" />
+    <gazebo reference="flipper_fl">
+        <material>Gazebo/Black</material>
+    </gazebo>
+    <gazebo reference="flipper_fr">
+        <material>Gazebo/Black</material>
+    </gazebo>
+    <gazebo reference="flipper_rl">
+        <material>Gazebo/Black</material>
+    </gazebo>
+    <gazebo reference="flipper_rr">
+        <material>Gazebo/Black</material>
+    </gazebo>
+    <gazebo reference="flipper_rr">
+        <material>Gazebo/Black</material>
+    </gazebo>
+    <gazebo reference="base_body">
+        <material>Gazebo/Red</material>
+    </gazebo>
     <gazebo>
         <plugin name="gazebo_ros_control" filename="libgazebo_ros_control.so">
@@ -58,7 +76,15 @@
             <robot_namespace>markhor</robot_namespace>
         </plugin>
-        <plugin filename="libKeysToCmdVelPlugin.so" name="keyboard_control">
-            <publish_as_twist>true</publish_as_twist>
-            <cmd_vel_topic>~/markhor/cmd_vel_twist</cmd_vel_topic>
+        <plugin name='tracked_vehicle_interface' filename='libgazebo_ros_tracked_vehicle_interface.so'>
+            <commandROSTopic>/cmd_vel</commandROSTopic>
+            <commandIGNTopic>~/markhor/cmd_vel_twist</commandIGNTopic>
+            <!-- <odometryTopic>~odom</odometryTopic> -->     <!-- ROS topic for the odometry data - remap if you're using another odom source -->
+            <!-- <trackSpeedTopic>~track_speed</trackSpeedTopic> -->  <!-- gazebo topic of SimpleTrackedVehicle -->
+            <robotBaseFrame>base_link</robotBaseFrame>
+            <!-- <odometryFrame>odom</odometryFrame> -->      <!-- tf frame of the odometry messages -->
+            <tracks_separation>${tracks_seperation}</tracks_separation>
+            <!--<publishOdomTF>true</publishOdomTF>  -->
+            <!--<updateRate>100.0</updateRate>  -->
+            <!-- <odometrySource>encoder</odometrySource> --> <!-- [encoder,world] - choose world for ground truth -->
         </plugin>
     </gazebo>

File: markhor_description/urdf/markhor_common.xacro (robot description, xacro)
@@ -70,5 +70,5 @@
             <type>transmission_interface/SimpleTransmission</type>
             <joint name="${flipper_name}_motor_j">
-                <hardwareInterface>hardware_interface/VelocityJointInterface</hardwareInterface>
+                <hardwareInterface>hardware_interface/EffortJointInterface</hardwareInterface>
             </joint>
             <actuator name="${flipper_name}_track_motor">
@@ -109,6 +109,6 @@
                     <horizontal_fov>1.047198</horizontal_fov>
                     <image>
-                        <width>640</width>
-                        <height>400</height>
+                        <width>1280</width>
+                        <height>720</height>
                         <format>R8G8B8</format>
                     </image>

Commit message: add tf_web_publisher

File: markhor_description/urdf/markhor.urdf.xacro (robot description, xacro)
@@ -10,4 +10,5 @@
     <link name="base_footprint" />
     <link name="base_link" />
+    <link name="markhor_link_base" />
     <link name="base_body">
         <visual>
@@ -29,4 +30,8 @@
         <parent link="base_link" />
         <child link="base_footprint" />
+    </joint>
+    <joint name="markhor_link_base_j" type="fixed">
+        <parent link="base_link" />
+        <child link="markhor_link_base" />
     </joint>
     <joint name="base_body_j" type="fixed">

Commit message: Implement Velodyne Radar

File: markhor_description/urdf/markhor.urdf.xacro (robot description, xacro)
@@ -1,5 +1,12 @@
 <?xml version="1.0"?>
 <robot xmlns:xacro="http://www.ros.org/wiki/xacro" name="markhor">
-    <xacro:include filename="$(find sick_tim)/urdf/sick_tim.urdf.xacro" />
+    <!--<xacro:include filename="$(find sick_tim)/urdf/sick_tim.urdf.xacro" />
+    <xacro:sick_tim551 name="laser" ros_topic="scan" />
+    <xacro:virtual_joint name="laser_mount_link" parent="base_link" origin_xyz="0.32034017 0 0.1393156" origin_rpy="0 0 0" />
+    -->
+    <xacro:include filename="$(find velodyne_description)/urdf/VLP-16.urdf.xacro" />
+    <xacro:VLP-16 name="laser" gpu="true">
+        <origin xyz="0.32034017 0 0.1393156" rpy="0 0 0" />
+    </xacro:VLP-16>
     <xacro:include filename="$(find markhor_description)/urdf/markhor_common.xacro" />
     <xacro:arg name="robot_namespace" default="markhor" />
@@ -46,6 +53,4 @@
     <xacro:camera_link link_name="rear_cam" camera_name="$(arg robot_namespace)/rear_cam" frame_name="rear_cam" parent="base_link" origin_xyz="-0.35864800 0 0.03810000" origin_rpy="0 0 ${pi}" />
     <xacro:virtual_anchor anchor_name="arm_root" parent="base_link" origin_xyz="0.17394875 0 0.12291060" origin_rpy="0 0 0" />
-    <xacro:sick_tim551 name="laser" ros_topic="scan" />
-    <xacro:virtual_joint name="laser_mount_link" parent="base_link" origin_xyz="0.32034017 0 0.1393156" origin_rpy="0 0 0" />
     <gazebo reference="flipper_fl">
         <material>Gazebo/Black</material>

Commit message: Add material colors for UI visualization

File: markhor_description/urdf/markhor.urdf.xacro (robot description, xacro)
@@ -20,4 +20,5 @@
             </geometry>
             <origin xyz="0 0 0" rpy="0 ${pi} 0" />
+            <material name="red"/>
         </visual>
         <collision>

File: markhor_description/urdf/markhor_common.xacro (robot description, xacro)
@@ -18,5 +18,5 @@
                 </geometry>
                 <origin xyz="0 0 0" rpy="0 0 0"/>
-                <material name="grey"/>
+                <material name="black"/>
             </visual>
             <collision>

Commit message: Boost up height, increase flipper torque

File: markhor_description/urdf/markhor.urdf.xacro (robot description, xacro)
@@ -9,5 +9,5 @@
     <xacro:property name="tracks_shift_x" value="0.31115000" />
     <xacro:property name="tracks_shift_y" value="0.2230283" />
-    <xacro:property name="tracks_height" value="0.05318760" />
+    <xacro:property name="tracks_height" value="0" />
     <xacro:property name="tracks_seperation" value="${tracks_shift_y} * 2" />
     <link name="base_footprint" />

File: markhor_description/urdf/markhor_common.xacro (robot description, xacro)
@@ -6,5 +6,5 @@
     <xacro:property name="flipper_upper_limit" value="0" />
     <xacro:property name="flipper_velocity_limit" value="16.75" />
-    <xacro:property name="flipper_torque_limit" value="184" />
+    <xacro:property name="flipper_torque_limit" value="1000" />
     <xacro:property name="track_velocity_limit" value="5.34" />
     <xacro:property name="track_torque_limit" value="94.5" />

Commit message: Update urdf with the new tower

File: markhor_description/urdf/markhor.urdf.xacro (robot description, xacro)
@@ -3,5 +3,5 @@
     <xacro:include filename="$(find velodyne_description)/urdf/VLP-16.urdf.xacro" />
     <xacro:VLP-16 name="laser" gpu="true">
-        <origin xyz="0.32034017 0 0.1393156" rpy="0 0 0" />
+        <origin xyz="-0.2875 0 0.45176" rpy="0 0 0" />
     </xacro:VLP-16>
     <xacro:include filename="$(find markhor_description)/urdf/markhor_common.xacro" />
@@ -13,5 +13,4 @@
     <link name="base_footprint" />
     <link name="base_link" />
-    <link name="markhor_link_base" />
     <link name="base_body">
         <visual>
@@ -30,12 +29,28 @@
         <xacro:markhor_inertial type="body" />
     </link>
+    <link name="tower_body">
+        <visual>
+            <geometry>
+                <mesh filename="package://markhor_description/meshes/LidarTower.stl" />
+            </geometry>
+            <origin xyz="0 0 0" rpy="0 0 -${pi/2}" />
+            <material name="grey"/>
+        </visual>
+        <collision>
+            <geometry>
+                <mesh filename="package://markhor_description/meshes/LidarTower.stl" />
+            </geometry>
+            <origin xyz="0 0 0" rpy="0 0 -${pi/2}" />
+        </collision>
+        <xacro:markhor_inertial type="body" />
+    </link>
+    <joint name="tower_body_j" type="fixed">
+        <parent link="base_link" />
+        <child link="tower_body" />
+    </joint>
     <joint name="base_link_j" type="fixed">
         <origin xyz="0 0 -0.085" rpy="0 0 0" />
         <parent link="base_link" />
         <child link="base_footprint" />
-    </joint>
-    <joint name="markhor_link_base_j" type="fixed">
-        <parent link="base_link" />
-        <child link="markhor_link_base" />
     </joint>
     <joint name="base_body_j" type="fixed">
@@ -49,22 +64,25 @@
     <xacro:camera_link link_name="front_cam" camera_name="$(arg robot_namespace)/front_cam" frame_name="front_cam" parent="base_link" origin_xyz="0.35864800 0 0.03810000" origin_rpy="0 0 0" />
     <xacro:camera_link link_name="rear_cam" camera_name="$(arg robot_namespace)/rear_cam" frame_name="rear_cam" parent="base_link" origin_xyz="-0.35864800 0 0.03810000" origin_rpy="0 0 ${pi}" />
-    <xacro:virtual_anchor anchor_name="arm_root" parent="base_link" origin_xyz="0.17394875 0 0.12291060" origin_rpy="0 0 0" />
+    <xacro:virtual_anchor anchor_name="arm_root" parent="base_link" origin_xyz="0.3 0 0.12291060" origin_rpy="0 0 0" />
     <gazebo reference="flipper_fl">
-        <material>Gazebo/Black</material>
+        <material>Gazebo/Grey</material>
     </gazebo>
     <gazebo reference="flipper_fr">
-        <material>Gazebo/Black</material>
+        <material>Gazebo/Grey</material>
     </gazebo>
     <gazebo reference="flipper_rl">
-        <material>Gazebo/Black</material>
+        <material>Gazebo/Grey</material>
     </gazebo>
     <gazebo reference="flipper_rr">
-        <material>Gazebo/Black</material>
+        <material>Gazebo/Grey</material>
     </gazebo>
     <gazebo reference="flipper_rr">
-        <material>Gazebo/Black</material>
+        <material>Gazebo/Grey</material>
     </gazebo>
     <gazebo reference="base_body">
         <material>Gazebo/Red</material>
+    </gazebo>
+    <gazebo reference="tower_body">
+        <material>Gazebo/Grey</material>
     </gazebo>
     <gazebo>

File: markhor_description/urdf/markhor_common.xacro (robot description, xacro)
@@ -18,5 +18,5 @@
                 </geometry>
                 <origin xyz="0 0 0" rpy="0 0 0"/>
-                <material name="black"/>
+                <material name="grey"/>
             </visual>
             <collision>

File: markhor_description/urdf/markhor_w_attachments.xacro (robot description, xacro)
@@ -5,6 +5,6 @@
   <xacro:include filename="$(find ovis_description)/urdf/ovis_standalone.xacro"/>
   <joint name="markhor_joint_fix_arm" type="fixed">
-    <origin rpy="${pi} ${pi} 0" xyz="0.17394875 0 0.12291060"/>
-    <parent link="base_link"/>
+    <origin rpy="${pi} ${pi} 0" xyz="0 0 0"/>
+    <parent link="arm_root"/>
     <child link="ovis_root"/>
   </joint>

Commit message: Rework tower to include new top

File: markhor_description/urdf/markhor.urdf.xacro (robot description, xacro)
@@ -3,5 +3,5 @@
     <xacro:include filename="$(find velodyne_description)/urdf/VLP-16.urdf.xacro" />
     <xacro:VLP-16 name="laser" gpu="true">
-        <origin xyz="-0.2875 0 0.45176" rpy="0 0 0" />
+        <origin xyz="-0.315 0 0.48" rpy="0 0 0" />
     </xacro:VLP-16>
     <xacro:include filename="$(find markhor_description)/urdf/markhor_common.xacro" />
@@ -32,14 +32,14 @@
         <visual>
             <geometry>
-                <mesh filename="package://markhor_description/meshes/LidarTower.stl" />
+                <mesh filename="package://markhor_description/meshes/tower.stl" />
             </geometry>
-            <origin xyz="0 0 0" rpy="0 0 -${pi/2}" />
+            <origin xyz="0 0 0" rpy="${pi/2} 0 0" />
             <material name="grey"/>
         </visual>
         <collision>
             <geometry>
-                <mesh filename="package://markhor_description/meshes/LidarTower.stl" />
+                <mesh filename="package://markhor_description/meshes/tower.stl" />
             </geometry>
-            <origin xyz="0 0 0" rpy="0 0 -${pi/2}" />
+            <origin xyz="0 0 0" rpy="${pi/2} 0 0" />
         </collision>
         <xacro:markhor_inertial type="body" />
@@ -48,4 +48,47 @@
         <parent link="base_link" />
         <child link="tower_body" />
+        <origin xyz="-0.314 0 .126" rpy="0 0 0" />
+    </joint>
+    <link name="tower_top">
+        <visual>
+            <geometry>
+                <mesh filename="package://markhor_description/meshes/tower_top.stl" />
+            </geometry>
+            <origin xyz="0 0 0" rpy="${pi/2} 0 0" />
+            <material name="grey"/>
+        </visual>
+        <collision>
+            <geometry>
+                <mesh filename="package://markhor_description/meshes/tower_top.stl" />
+            </geometry>
+            <origin xyz="0 0 0" rpy="${pi/2} 0 0" />
+        </collision>
+        <xacro:markhor_inertial type="body" />
+    </link>
+    <joint name="tower_top_j" type="fixed">
+        <parent link="tower_body" />
+        <child link="tower_top" />
+        <origin xyz="0 0 .44" rpy="0 0 0" />
+    </joint>
+    <link name="tpv_base">
+        <visual>
+            <geometry>
+                <mesh filename="package://markhor_description/meshes/TPV_base.stl" />
+            </geometry>
+            <origin xyz="0 0 0" rpy="${pi/2} 0 0" />
+            <material name="grey"/>
+        </visual>
+        <collision>
+            <geometry>
+                <mesh filename="package://markhor_description/meshes/TPV_base.stl" />
+            </geometry>
+            <origin xyz="0 0 0" rpy="${pi/2} 0 0" />
+        </collision>
+        <xacro:markhor_inertial type="body" />
+    </link>
+    <joint name="tpv_base_j" type="fixed">
+        <parent link="tower_top" />
+        <child link="tpv_base" />
+        <origin xyz="0 0 .02" rpy="0 0 0" />
     </joint>
     <joint name="base_link_j" type="fixed">

Commit message: add base joint, separate tower in a new file

File: markhor_description/urdf/markhor.urdf.xacro (robot description, xacro)
@@ -1,9 +1,6 @@
 <?xml version="1.0"?>
 <robot xmlns:xacro="http://www.ros.org/wiki/xacro" name="markhor">
-    <xacro:include filename="$(find velodyne_description)/urdf/VLP-16.urdf.xacro" />
-    <xacro:VLP-16 name="laser" gpu="true">
-        <origin xyz="-0.315 0 0.48" rpy="0 0 0" />
-    </xacro:VLP-16>
     <xacro:include filename="$(find markhor_description)/urdf/markhor_common.xacro" />
+    <xacro:include filename="$(find markhor_description)/urdf/tower.xacro" />
     <xacro:arg name="robot_namespace" default="markhor" />
     <xacro:property name="tracks_shift_x" value="0.31115000" />
@@ -29,67 +26,4 @@
         <xacro:markhor_inertial type="body" />
     </link>
-    <link name="tower_body">
-        <visual>
-            <geometry>
-                <mesh filename="package://markhor_description/meshes/tower.stl" />
-            </geometry>
-            <origin xyz="0 0 0" rpy="${pi/2} 0 0" />
-            <material name="grey"/>
-        </visual>
-        <collision>
-            <geometry>
-                <mesh filename="package://markhor_description/meshes/tower.stl" />
-            </geometry>
-            <origin xyz="0 0 0" rpy="${pi/2} 0 0" />
-        </collision>
-        <xacro:markhor_inertial type="body" />
-    </link>
-    <joint name="tower_body_j" type="fixed">
-        <parent link="base_link" />
-        <child link="tower_body" />
-        <origin xyz="-0.314 0 .126" rpy="0 0 0" />
-    </joint>
-    <link name="tower_top">
-        <visual>
-            <geometry>
-                <mesh filename="package://markhor_description/meshes/tower_top.stl" />
-            </geometry>
-            <origin xyz="0 0 0" rpy="${pi/2} 0 0" />
-            <material name="grey"/>
-        </visual>
-        <collision>
-            <geometry>
-                <mesh filename="package://markhor_description/meshes/tower_top.stl" />
-            </geometry>
-            <origin xyz="0 0 0" rpy="${pi/2} 0 0" />
-        </collision>
-        <xacro:markhor_inertial type="body" />
-    </link>
-    <joint name="tower_top_j" type="fixed">
-        <parent link="tower_body" />
-        <child link="tower_top" />
-        <origin xyz="0 0 .44" rpy="0 0 0" />
-    </joint>
-    <link name="tpv_base">
-        <visual>
-            <geometry>
-                <mesh filename="package://markhor_description/meshes/TPV_base.stl" />
-            </geometry>
-            <origin xyz="0 0 0" rpy="${pi/2} 0 0" />
-            <material name="grey"/>
-        </visual>
-        <collision>
-            <geometry>
-                <mesh filename="package://markhor_description/meshes/TPV_base.stl" />
-            </geometry>
-            <origin xyz="0 0 0" rpy="${pi/2} 0 0" />
-        </collision>
-        <xacro:markhor_inertial type="body" />
-    </link>
-    <joint name="tpv_base_j" type="fixed">
-        <parent link="tower_top" />
-        <child link="tpv_base" />
-        <origin xyz="0 0 .02" rpy="0 0 0" />
-    </joint>
     <joint name="base_link_j" type="fixed">
         <origin xyz="0 0 -0.085" rpy="0 0 0" />
