Commit message: Add tilt axis and Zed

File: markhor_description/urdf/tower.xacro (robot description, xacro)
@@ -1,4 +1,12 @@
 <?xml version="1.0"?>
 <root xmlns:xi="http://www.w3.org/2001/XInclude" xmlns:xacro="http://www.ros.org/wiki/xacro">
+    <xacro:include filename="$(find zed_wrapper)/urdf/zed_macro.urdf.xacro" />
+    <xacro:zed_camera name="zed2" model="zed2" parent="tpv_tilt">
+        <origin xyz="0 0 -0.0125" rpy="0 0 0"/>
+    </xacro:zed_camera>
+    <xacro:include filename="$(find velodyne_description)/urdf/VLP-16.urdf.xacro" />
+    <xacro:VLP-16 name="laser" gpu="true" parent="tower_body">
+        <origin xyz="0 0 0.355" rpy="0 0 0" />
+    </xacro:VLP-16>
     <link name="tower_body">
         <visual>
@@ -22,8 +30,4 @@
         <origin xyz="-0.314 0 .126" rpy="0 0 0" />
     </joint>
-    <xacro:include filename="$(find velodyne_description)/urdf/VLP-16.urdf.xacro" />
-    <xacro:VLP-16 name="laser" gpu="true" parent="tower_body">
-        <origin xyz="0 0 0.355" rpy="0 0 0" />
-    </xacro:VLP-16>
     <link name="tower_top">
         <visual>
@@ -69,3 +73,23 @@
         <origin xyz="0 0 .01" rpy="0 0 0" />
     </joint>
+    <transmission name="tpv_base_trans">
+        <type>transmission_interface/SimpleTransmission</type>
+        <joint name="tpv_base_j">
+            <hardwareInterface>PositionJointInterface</hardwareInterface>
+        </joint>
+        <actuator name="tpv_base_motor"/>
+    </transmission>
+    <link name="tpv_tilt_axis"/>
+    <joint name="tpv_tilt_axis_j" type="fixed">
+        <parent link="tpv_base" />
+        <child link="tpv_tilt_axis" />
+        <origin xyz=".065 0 .045" rpy="0 0 0" />
+    </joint>
+    <link name="tpv_tilt"/>
+    <joint name="tpv_tilt_j" type="continuous">
+        <parent link="tpv_tilt_axis" />
+        <child link="tpv_tilt" />
+        <axis xyz="0 1 0"/>
+        <origin xyz="0 0 0" rpy="0 0 0" />
+    </joint>
 </root>

Commit message: Add tilt carriage 3d model

File: markhor_description/urdf/tower.xacro (robot description, xacro)
@@ -3,5 +3,5 @@
     <xacro:include filename="$(find zed_wrapper)/urdf/zed_macro.urdf.xacro" />
     <xacro:zed_camera name="zed2" model="zed2" parent="tpv_tilt">
-        <origin xyz="0 0 -0.0125" rpy="0 0 0"/>
+        <origin xyz="0.015 0 -0.0125" rpy="0 0 0"/>
     </xacro:zed_camera>
     <xacro:include filename="$(find velodyne_description)/urdf/VLP-16.urdf.xacro" />
@@ -86,5 +86,20 @@
         <origin xyz=".065 0 .045" rpy="0 0 0" />
     </joint>
-    <link name="tpv_tilt"/>
+    <link name="tpv_tilt">
+        <visual>
+            <geometry>
+                <mesh filename="package://markhor_description/meshes/tpv_tilt.stl" />
+            </geometry>
+            <origin xyz="0 0 0" rpy="${pi/2} 0 ${pi/2}" />
+            <material name="grey"/>
+        </visual>
+        <collision>
+            <geometry>
+                <mesh filename="package://markhor_description/meshes/tpv_tilt.stl" />
+            </geometry>
+            <origin xyz="0 0 0" rpy="${pi/2} 0 ${pi/2}" />
+        </collision>
+        <xacro:markhor_inertial type="body" />
+    </link>
     <joint name="tpv_tilt_j" type="continuous">
         <parent link="tpv_tilt_axis" />

Commit message: Add tilt axis transmission (for future gazebo use)

File: markhor_description/urdf/tower.xacro (robot description, xacro)
@@ -108,3 +108,10 @@
         <origin xyz="0 0 0" rpy="0 0 0" />
     </joint>
+    <transmission name="tpv_tilt_trans">
+        <type>transmission_interface/SimpleTransmission</type>
+        <joint name="tpv_tilt_j">
+            <hardwareInterface>PositionJointInterface</hardwareInterface>
+        </joint>
+        <actuator name="tpv_tilt_motor"/>
+    </transmission>
 </root>

Commit message: add env var to tower

File: markhor_description/urdf/tower.xacro (robot description, xacro)
@@ -1,8 +1,12 @@
 <?xml version="1.0"?>
 <root xmlns:xi="http://www.w3.org/2001/XInclude" xmlns:xacro="http://www.ros.org/wiki/xacro">
-    <xacro:include filename="$(find zed_wrapper)/urdf/zed_macro.urdf.xacro" />
-    <xacro:zed_camera name="zed2" model="zed2" parent="tpv_tilt">
+    <!-- Get the ENV simulation variable (default to false) -->
+    <xacro:property name="simulation" value="$(optenv simulation false)"/>
+    <xacro:if value="${not simulation}">
+        <xacro:include filename="$(find zed_wrapper)/urdf/zed_macro.urdf.xacro" />
+        <xacro:zed_camera name="zed2" model="zed2" parent="tpv_tilt">
         <origin xyz="0.015 0 -0.0125" rpy="0 0 0"/>
-    </xacro:zed_camera>
+        </xacro:zed_camera>
+    </xacro:if>
     <xacro:include filename="$(find velodyne_description)/urdf/VLP-16.urdf.xacro" />
     <xacro:VLP-16 name="laser" gpu="true" parent="tower_body">

Commit message: add env variable for gui gazebo

File: markhor_description/urdf/tower.xacro (robot description, xacro)
@@ -2,5 +2,5 @@
 <root xmlns:xi="http://www.w3.org/2001/XInclude" xmlns:xacro="http://www.ros.org/wiki/xacro">
     <!-- Get the ENV simulation variable (default to false) -->
-    <xacro:property name="simulation" value="$(optenv simulation false)"/>
+    <xacro:property name="simulation" value="$(optenv MARKHOR_SIMULATION false)"/>
     <xacro:if value="${not simulation}">
         <xacro:include filename="$(find zed_wrapper)/urdf/zed_macro.urdf.xacro" />

Commit message: reapply changes from ftr/docker

File: markhor_description/urdf/tower.xacro (robot description, xacro)
@@ -1,8 +1,12 @@
 <?xml version="1.0"?>
 <root xmlns:xi="http://www.w3.org/2001/XInclude" xmlns:xacro="http://www.ros.org/wiki/xacro">
-    <xacro:include filename="$(find zed_wrapper)/urdf/zed_macro.urdf.xacro" />
-    <xacro:zed_camera name="zed2" model="zed2" parent="tpv_tilt">
+    <!-- Get the ENV simulation variable (default to false) -->
+    <xacro:property name="simulation" value="$(optenv MARKHOR_SIMULATION false)"/>
+    <xacro:if value="${not simulation}">
+        <xacro:include filename="$(find zed_wrapper)/urdf/zed_macro.urdf.xacro" />
+        <xacro:zed_camera name="zed2" model="zed2" parent="tpv_tilt">
         <origin xyz="0.015 0 -0.0125" rpy="0 0 0"/>
-    </xacro:zed_camera>
+        </xacro:zed_camera>
+    </xacro:if>
     <xacro:include filename="$(find velodyne_description)/urdf/VLP-16.urdf.xacro" />
     <xacro:VLP-16 name="laser" gpu="true" parent="tower_body">

Commit message: fix flipper appearance in rviz

File: markhor_description/urdf/tower.xacro (robot description, xacro)
@@ -112,10 +112,3 @@
         <origin xyz="0 0 0" rpy="0 0 0" />
     </joint>
-    <transmission name="tpv_tilt_trans">
-        <type>transmission_interface/SimpleTransmission</type>
-        <joint name="tpv_tilt_j">
-            <hardwareInterface>PositionJointInterface</hardwareInterface>
-        </joint>
-        <actuator name="tpv_tilt_motor"/>
-    </transmission>
 </root>

Commit message: change velodyne transform to match urdf

File: markhor_description/urdf/tower.xacro (robot description, xacro)
@@ -13,4 +13,10 @@
         <origin xyz="0 0 0.355" rpy="0 0 0" />
     </xacro:VLP-16>
+    <link name="velodyne"/>
+    <joint name="velodyne_j" type="fixed">
+        <parent link="tower_body" />
+        <child link="velodyne" />
+        <origin xyz="0 0 0.355" rpy="0 0 0" />
+    </joint>
     <link name="tower_body">
         <visual>
